File: Orthodox.kicad_pcb (KiCad board)
At the start: 2 copper layers, 252.6 x 100.2 mm, 121 parts, among them SW1 SW_Push, SW10 SW_Push, SW11 SW_Push, SW12 SW_Push, SW13 SW_Push, SW14 SW_Push, SW15 SW_Push, SW16 SW_Push, SW17 SW_Push, SW18 SW_Push, SW19 SW_Push, SW2 SW_Push, SW20 SW_Push, SW21 SW_Push, SW22 SW_Push, SW23 SW_Push, SW24 SW_Push, SW25 SW_Push, SW26 SW_Push, SW27 SW_Push, SW28 SW_Push, SW29 SW_Push, SW3 SW_Push, SW30 SW_Push, SW31 SW_Push, SW32 SW_Push, SW33 SW_Push, SW34 SW_Push, SW35 SW_Push, SW36 SW_Push, SW37 SW_Push, SW38 SW_Push, SW39 SW_Push, SW4 SW_Push, SW40 RED, SW41 SW_Push, SW42 SW_Push, SW43 SW_Push, SW44 SW_Push, SW45 SW_Push, SW46 SW_Push, SW47 SW_Push, SW48 SW_Push, SW49 SW_Push, SW5 SW_Push, SW50 SW_Push, SW51 SW_Push, SW52 SW_Push, SW53 BLUE, SW54 GREEN, SW55 SW_Push, SW56 SW_Push, SW57 SW_Push, SW58 SW_Push, SW59 SW_Push, SW6 SW_Push, SW60 SW_Push, SW7 SW_Push, SW8 SW_Push, SW9 SW_Push, U1 ATmega32U4-AU

Commit message: Updated to V6 and used fillets
Parts:
- SW40, SW53, SW54: footprint Switch_Keyboard_Kailh:SW_58_Series_Kalih_Reduced -> Switch_Keyboard_Kailh:SW_58_Series_Kalih
Connections:
- U1 pad 1: Net-(U1-Pad1) -> unconnected-(U1-Pad1)
- U1 pad 10: Net-(U1-Pad10) -> unconnected-(U1-Pad10)
- U1 pad 11: Net-(U1-Pad11) -> unconnected-(U1-Pad11)
- U1 pad 12: Net-(U1-Pad12) -> unconnected-(U1-Pad12)
- U1 pad 13: Net-(U1-Pad13) -> unconnected-(U1-Pad13)
- U1 pad 16: Net-(U1-Pad16) -> unconnected-(U1-Pad16)
- U1 pad 17: Net-(U1-Pad17) -> unconnected-(U1-Pad17)
- U1 pad 18: Net-(U1-Pad18) -> unconnected-(U1-Pad18)
- U1 pad 19: Net-(U1-Pad19) -> unconnected-(U1-Pad19)
- U1 pad 2: Net-(U1-Pad2) -> unconnected-(U1-Pad2)
- U1 pad 20: Net-(U1-Pad20) -> unconnected-(U1-Pad20)
- U1 pad 21: Net-(U1-Pad21) -> unconnected-(U1-Pad21)
- U1 pad 22: Net-(U1-Pad22) -> unconnected-(U1-Pad22)
- U1 pad 25: Net-(U1-Pad25) -> unconnected-(U1-Pad25)
- U1 pad 26: Net-(U1-Pad26) -> unconnected-(U1-Pad26)
- U1 pad 27: Net-(U1-Pad27) -> unconnected-(U1-Pad27)
- U1 pad 28: Net-(U1-Pad28) -> unconnected-(U1-Pad28)
- U1 pad 29: Net-(U1-Pad29) -> unconnected-(U1-Pad29)
- U1 pad 3: Net-(U1-Pad3) -> unconnected-(U1-Pad3)
- U1 pad 30: Net-(U1-Pad30) -> unconnected-(U1-Pad30)
- U1 pad 31: Net-(U1-Pad31) -> unconnected-(U1-Pad31)
- U1 pad 32: Net-(U1-Pad32) -> unconnected-(U1-Pad32)
- U1 pad 33: Net-(U1-Pad33) -> unconnected-(U1-Pad33)
- U1 pad 36: Net-(U1-Pad36) -> unconnected-(U1-Pad36)
- U1 pad 37: Net-(U1-Pad37) -> unconnected-(U1-Pad37)
- U1 pad 38: Net-(U1-Pad38) -> unconnected-(U1-Pad38)
- U1 pad 39: Net-(U1-Pad39) -> unconnected-(U1-Pad39)
- U1 pad 4: Net-(U1-Pad4) -> unconnected-(U1-Pad4)
- U1 pad 40: Net-(U1-Pad40) -> unconnected-(U1-Pad40)
- U1 pad 41: Net-(U1-Pad41) -> unconnected-(U1-Pad41)
- U1 pad 42: Net-(U1-Pad42) -> unconnected-(U1-Pad42)
- U1 pad 5: Net-(U1-Pad5) -> unconnected-(U1-Pad5)
- U1 pad 6: Net-(U1-Pad6) -> unconnected-(U1-Pad6)
- U1 pad 7: Net-(U1-Pad7) -> unconnected-(U1-Pad7)
- U1 pad 8: Net-(U1-Pad8) -> unconnected-(U1-Pad8)
- U1 pad 9: Net-(U1-Pad9) -> unconnected-(U1-Pad9)
Routing:
- net COL12: track 208.4 -> 242.7 mm
- net ROW6: track 315.3 -> 348.0 mm
- net COL11: track 183.0 -> 208.4 mm
- net ROW4: track 319.1 -> 344.3 mm
- net COL4: track 85.5 -> 61.1 mm
- net COL5: track 84.3 -> 61.1 mm
- net ROW3: track 367.6 -> 390.7 mm
- net ROW1: track 372.7 -> 394.2 mm
- net ROW0: track 406.1 -> 424.2 mm
- net COL9: track 155.8 -> 170.9 mm
- net COL8: track 130.5 -> 143.0 mm
- net COL10: track 177.1 -> 189.2 mm
- net COL0: track 185.9 -> 196.4 mm
- net COL7: track 112.3 -> 119.8 mm
- net COL2: track 125.4 -> 123.1 mm
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Other:
- net class Default removed
- net class Large removed

Commit message: Half way through cleaning up keyswitch models and placement
Parts:
- D1, D10, D11, D12, D13, D14, D15, D16, D17, D18, D19, D2, D20, D21, D22, D23, D24, D25, D26, D27, D28, D29, D3, D30, D31, D32, D33, D34, D35, D36, D37, D38, D39, D4, D40, D41, D42, D43, D44, D45, D46, D47, D48, D49, D5, D50, D51, D52, D53, D54, D55, D56, D57, D58, D59, D6, D60, D7, D8, D9: footprint Diode_SMD:D_1206_3216Metric_Pad1.42x1.75mm_HandSolder -> Diode_SMD:D_1206_3216Metric
- U1: value ATmega32U4-AU -> AT90USB1286-A; footprint Package_QFP:TQFP-44_10x10mm_P0.8mm -> Package_QFP:TQFP-64_14x14mm_P0.8mm
- moved U1 36.5 mm to (201.8, 199.5), turned to 0 degrees
- moved D9 5.12 mm to (116.3, 143.8)
- moved D10 5.01 mm to (106.8, 153.3)
- moved D15 5.00 mm to (116.3, 153.3)
- moved D1 0.68 mm to (97.2, 86.6)
- moved SW54 0.65 mm to (116.1, 156.6)
- moved SW53 0.64 mm to (106.5, 156.6)
- moved D13 0.59 mm to (135.3, 124.7)
- moved D18 0.59 mm to (154.4, 124.7)
- moved D23 0.59 mm to (173.4, 124.7)
- moved D28 0.59 mm to (192.5, 124.7)
- moved D3 0.59 mm to (97.2, 124.7)
- moved D32 0.59 mm to (211.6, 124.7)
- moved D36 0.59 mm to (230.6, 124.7)
- moved D40 0.59 mm to (249.7, 124.7)
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Connections:
- U1 pad 14: Net-(U1-Pad14) -> unconnected-(U1-Pad14)
- U1 pad 15: Net-(U1-Pad15) -> unconnected-(U1-Pad15)
- U1 pad 21: unconnected-(U1-Pad21) -> Net-(U1-Pad21)
- U1 pad 22: unconnected-(U1-Pad22) -> Net-(U1-Pad22)
- U1 pad 23: Net-(U1-Pad15) -> unconnected-(U1-Pad23)
- U1 pad 24: Net-(U1-Pad24) -> unconnected-(U1-Pad24)
- U1 pad 34: Net-(U1-Pad14) -> unconnected-(U1-Pad34)
- U1 pad 35: Net-(U1-Pad15) -> unconnected-(U1-Pad35)
- U1 pad 43: Net-(U1-Pad15) -> unconnected-(U1-Pad43)
- U1 pad 44: Net-(U1-Pad24) -> unconnected-(U1-Pad44)
Routing:
- net ROW3: track 390.7 -> 77.9 mm
- net ROW1: track 394.2 -> 100.4 mm
- net ROW6: track 348.0 -> 68.9 mm
- net ROW4: track 344.3 -> 68.0 mm
- net ROW0: track 424.2 -> 177.2 mm
- net ROW5: track 9.53 -> 0.00 mm
- net Net-(D10-Pad2): track 4.31 -> 0.00 mm
- net Net-(D9-Pad2): track 4.22 -> 0.00 mm
- net Net-(D15-Pad2): track 4.17 -> 0.00 mm
- net Net-(D60-Pad2): track 3.52 -> 0.00 mm
- net Net-(D55-Pad2): track 3.52 -> 0.00 mm
- net Net-(D54-Pad2): track 3.52 -> 0.00 mm
- net Net-(D59-Pad2): track 3.52 -> 0.00 mm
- net Net-(D5-Pad2): track 3.52 -> 0.00 mm
- net Net-(D41-Pad2): track 3.52 -> 0.00 mm
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Other:
- board size 252.6 x 100.2 mm -> 252.7 x 100.5 mm

Commit message: Cleaned up
Parts:
- moved D11 0.64 mm to (135.3, 86.6)
- moved D16 0.64 mm to (154.4, 86.6)
- moved D21 0.64 mm to (173.4, 86.6)
- moved D26 0.64 mm to (192.5, 86.6)
- moved D30 0.64 mm to (211.6, 86.6)
- moved D34 0.64 mm to (230.6, 86.6)
- moved D38 0.64 mm to (249.7, 86.6)
- moved D42 0.64 mm to (268.7, 86.6)
- moved D47 0.64 mm to (287.8, 86.6)
- moved D52 0.64 mm to (306.8, 86.6)
- moved D56 0.64 mm to (325.9, 86.6)
- moved D6 0.64 mm to (116.3, 86.6)
- moved D57 0.64 mm to (316.3, 105.6)
- moved D12 0.62 mm to (135.3, 105.6)
- moved D17 0.62 mm to (154.4, 105.6)
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Routing:
- net ROW3: track 77.9 -> 312.5 mm
- net ROW1: track 100.4 -> 316.7 mm
- net ROW4: track 68.0 -> 265.1 mm
- net ROW6: track 68.9 -> 263.1 mm
- net ROW0: track 177.2 -> 347.1 mm
- net Net-(D6-Pad2): track 0.00 -> 2.96 mm
- net Net-(D56-Pad2): track 0.00 -> 2.96 mm
- net Net-(D52-Pad2): track 0.00 -> 2.96 mm
- net Net-(D47-Pad2): track 0.00 -> 2.96 mm
- net Net-(D42-Pad2): track 0.00 -> 2.96 mm
- net Net-(D38-Pad2): track 0.00 -> 2.96 mm
- net Net-(D34-Pad2): track 0.00 -> 2.96 mm
- net Net-(D30-Pad2): track 0.00 -> 2.96 mm
- net Net-(D26-Pad2): track 0.00 -> 2.96 mm
- net Net-(D21-Pad2): track 0.00 -> 2.96 mm
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Other:
- board size 252.7 x 100.5 mm -> 252.7 x 100.3 mm

Commit message: Cleanup, reference designs and sticking with atmega
Parts:
- added C1: C, Capacitor_SMD:C_0603_1608Metric, B.Cu at (184.1, 165.3)
- added C2: 22p, Capacitor_SMD:C_0603_1608Metric, B.Cu at (188.1, 172.6)
- added C3: 22p, Capacitor_SMD:C_0603_1608Metric, B.Cu at (182.1, 178.6)
- added C4: C, Capacitor_SMD:C_0603_1608Metric, B.Cu at (174.1, 164.1)
- added C5: C, Capacitor_SMD:C_0603_1608Metric, B.Cu at (175.2, 160.8)
- added C6: C, Capacitor_SMD:C_0603_1608Metric, B.Cu at (176.3, 161.9)
- added C7: C, Capacitor_SMD:C_0603_1608Metric, B.Cu at (173.0, 162.9)
- added J1: USB_C_Receptacle_USB2.0, USB:GCT_USB4055-30-A, B.Cu at (180.4, 85.2)
- added R1: 10k, Resistor_SMD:R_0603_1608Metric, B.Cu at (185.2, 166.4)
- added R2: 10k, Resistor_SMD:R_0603_1608Metric, B.Cu at (169.0, 172.6)
- added R3: 22R, Resistor_SMD:R_0603_1608Metric, B.Cu at (183.0, 164.2)
- added R4: 22R, Resistor_SMD:R_0603_1608Metric, B.Cu at (181.8, 163.1)
- added SW61: SW_Push, Button_Switch_SMD:Panasonic_EVQPUJ_EVQPUA, B.Cu at (189.8, 168.4)
- added Y1: Crystal_GND24, Crystal:Crystal_SMD_0603-4Pin_6.0x3.5mm, B.Cu at (185.6, 176.0)
- U1: value AT90USB1286-A -> ATmega32U4-A; footprint Package_QFP:TQFP-64_14x14mm_P0.8mm -> Package_QFP:TQFP-44_10x10mm_P0.8mm; moved to B.Cu
- moved U1 37.2 mm to (178.0, 170.9), turned to -135 degrees
Connections:
- D10 pad 1: ROW5 -> ROW4
- D13 pad 1: ROW3 -> ROW2
- D14 pad 1: ROW4 -> ROW3
- D15 pad 1: ROW5 -> ROW4
- D18 pad 1: ROW3 -> ROW2
- D19 pad 1: ROW4 -> ROW3
- D20 pad 1: ROW6 -> ROW5
- D23 pad 1: ROW3 -> ROW2
- D24 pad 1: ROW4 -> ROW3
- D25 pad 1: ROW6 -> ROW5
- D28 pad 1: ROW3 -> ROW2
- D29 pad 1: ROW4 -> ROW3
- D3 pad 1: ROW3 -> ROW2
- D32 pad 1: ROW3 -> ROW2
- D33 pad 1: ROW4 -> ROW3
- D36 pad 1: ROW3 -> ROW2
- D37 pad 1: ROW4 -> ROW3
- D4 pad 1: ROW4 -> ROW3
- D40 pad 1: ROW3 -> ROW2
- D41 pad 1: ROW4 -> ROW3
- D44 pad 1: ROW3 -> ROW2
- D45 pad 1: ROW4 -> ROW3
- D46 pad 1: ROW6 -> ROW5
- D49 pad 1: ROW3 -> ROW2
- D5 pad 1: ROW6 -> ROW5
- D50 pad 1: ROW4 -> ROW3
- D51 pad 1: ROW6 -> ROW5
- D53 pad 1: ROW3 -> ROW2
- D54 pad 1: ROW4 -> ROW3
- D55 pad 1: ROW6 -> ROW5
- D58 pad 1: ROW3 -> ROW2
- D59 pad 1: ROW6 -> ROW5
- D60 pad 1: ROW6 -> ROW5
- D8 pad 1: ROW3 -> ROW2
- D9 pad 1: ROW4 -> ROW3
- U1 pad 1: unconnected-(U1-Pad1) -> ROW0
- U1 pad 10: unconnected-(U1-Pad10) -> MOSI
- U1 pad 11: unconnected-(U1-Pad11) -> MISO
- U1 pad 12: unconnected-(U1-Pad12) -> COL6
- U1 pad 13: unconnected-(U1-Pad13) -> Reset
- U1 pad 14: unconnected-(U1-Pad14) -> +5V
- U1 pad 15: unconnected-(U1-Pad15) -> GND
- U1 pad 16: unconnected-(U1-Pad16) -> XTAL2
- U1 pad 17: unconnected-(U1-Pad17) -> XTAL1
- U1 pad 19: unconnected-(U1-Pad19) -> COL3
- U1 pad 2: unconnected-(U1-Pad2) -> +5V
- U1 pad 21: Net-(U1-Pad21) -> unconnected-(U1-Pad21)
- U1 pad 22: Net-(U1-Pad22) -> COL11
- U1 pad 23: unconnected-(U1-Pad23) -> GND
- U1 pad 24: unconnected-(U1-Pad24) -> +5V
- U1 pad 25: unconnected-(U1-Pad25) -> COL10
- U1 pad 26: unconnected-(U1-Pad26) -> COL9
- U1 pad 27: unconnected-(U1-Pad27) -> COL8
- U1 pad 28: unconnected-(U1-Pad28) -> ROW5
- U1 pad 29: unconnected-(U1-Pad29) -> ROW1
- U1 pad 3: unconnected-(U1-Pad3) -> Net-(U1-Pad3)
- U1 pad 30: unconnected-(U1-Pad30) -> COL7
- U1 pad 31: unconnected-(U1-Pad31) -> COL5
- U1 pad 32: unconnected-(U1-Pad32) -> COL4
- U1 pad 33: unconnected-(U1-Pad33) -> Net-(U1-Pad33)
- U1 pad 34: unconnected-(U1-Pad34) -> +5V
- U1 pad 35: unconnected-(U1-Pad35) -> GND
- U1 pad 36: unconnected-(U1-Pad36) -> ROW2
- U1 pad 37: unconnected-(U1-Pad37) -> COL0
- U1 pad 38: unconnected-(U1-Pad38) -> ROW4
- U1 pad 39: unconnected-(U1-Pad39) -> ROW3
- U1 pad 4: unconnected-(U1-Pad4) -> Net-(U1-Pad4)
- U1 pad 40: unconnected-(U1-Pad40) -> COL2
- U1 pad 43: unconnected-(U1-Pad43) -> GND
- U1 pad 44: unconnected-(U1-Pad44) -> +5V
- U1 pad 5: unconnected-(U1-Pad5) -> GND
- U1 pad 6: unconnected-(U1-Pad6) -> Net-(C1-Pad1)
- U1 pad 7: unconnected-(U1-Pad7) -> +5V
- U1 pad 8: unconnected-(U1-Pad8) -> COL1
- U1 pad 9: unconnected-(U1-Pad9) -> SCK
Routing:
- net ROW2: track 0.00 -> 312.6 mm, vias 0 -> 2
- net ROW4: track 265.1 -> 0.00 mm
- net ROW5: track 0.00 -> 263.2 mm, vias 0 -> 2
- net ROW6: track 263.1 -> 0.00 mm
- net +5V: track 0.00 -> 92.1 mm
- net GND: track 0.00 -> 77.2 mm
- net D+: track 0.00 -> 76.0 mm
- net D-: track 0.00 -> 73.5 mm
- net ROW3: track 312.5 -> 265.2 mm, vias 0 -> 2
- net COL3: track 94.8 -> 121.0 mm
- net Reset: track 0.00 -> 8.09 mm
- net COL1: track 142.4 -> 148.1 mm
- net Net-(D10-Pad2): track 0.00 -> 3.93 mm
- net Net-(D15-Pad2): track 0.00 -> 3.92 mm
- net Net-(D9-Pad2): track 0.00 -> 3.92 mm
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- added copper zone on B.Cu, net +5V
- added copper zone on B.Cu, net GND
- added copper zone on F.Cu, net GND

Commit message: Rought placement of mounting holes + routing
Parts:
- moved C3 0.05 mm to (182.1, 178.5)
Connections:
- D20 pad 1: ROW5 -> ROW4
- D25 pad 1: ROW5 -> ROW4
- D46 pad 1: ROW5 -> ROW4
- D5 pad 1: ROW5 -> ROW4
- D51 pad 1: ROW5 -> ROW4
- D55 pad 1: ROW5 -> ROW4
- D59 pad 1: ROW5 -> ROW4
- D60 pad 1: ROW5 -> ROW4
- U1 pad 1: ROW0 -> unconnected-(U1-Pad1)
- U1 pad 12: COL6 -> COL7
- U1 pad 18: unconnected-(U1-Pad18) -> COL8
- U1 pad 19: COL3 -> COL9
- U1 pad 20: unconnected-(U1-Pad20) -> COL10
- U1 pad 21: unconnected-(U1-Pad21) -> COL11
- U1 pad 22: COL11 -> COL12
- U1 pad 25: COL10 -> ROW0
- U1 pad 26: COL9 -> ROW1
- U1 pad 27: COL8 -> ROW2
- U1 pad 28: ROW5 -> ROW3
- U1 pad 29: ROW1 -> ROW4
- U1 pad 30: COL7 -> COL0
- U1 pad 31: COL5 -> COL1
- U1 pad 32: COL4 -> COL2
- U1 pad 36: ROW2 -> COL3
- U1 pad 37: COL0 -> COL4
- U1 pad 38: ROW4 -> unconnected-(U1-Pad38)
- U1 pad 39: ROW3 -> unconnected-(U1-Pad39)
- U1 pad 40: COL2 -> unconnected-(U1-Pad40)
- U1 pad 41: unconnected-(U1-Pad41) -> COL6
- U1 pad 8: COL1 -> COL5
Routing:
- net ROW4: track 0.00 -> 372.5 mm, vias 0 -> 2
- net ROW5: track 263.2 -> 0.00 mm, vias 2 -> 0
- net ROW1: track 316.7 -> 401.7 mm
- net ROW2: track 312.6 -> 396.8 mm
- net ROW0: track 347.5 -> 431.5 mm
- net ROW3: track 265.2 -> 348.8 mm
- net COL5: track 60.9 -> 89.5 mm, vias 0 -> 1
- net +5V: track 92.1 -> 117.0 mm
- net COL2: track 122.2 -> 143.3 mm, vias 0 -> 1
- net COL1: track 148.1 -> 169.1 mm, vias 0 -> 1
- net COL10: track 189.2 -> 205.7 mm, vias 0 -> 1
- net COL7: track 119.8 -> 135.9 mm, vias 0 -> 1
- net COL9: track 170.9 -> 186.6 mm, vias 0 -> 1
- net COL8: track 143.0 -> 158.7 mm, vias 0 -> 1
- net COL0: track 197.7 -> 212.7 mm, vias 0 -> 1
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- removed copper zone on B.Cu, net +5V
Other:
- board size 252.7 x 100.3 mm -> 253.2 x 100.8 mm
