File: Orthodox.kicad_sch (KiCad schematic)
At the start: 121 parts, among them SW1 SW_Push, SW10 SW_Push, SW11 SW_Push, SW12 SW_Push, SW13 SW_Push, SW14 SW_Push, SW15 SW_Push, SW16 SW_Push, SW17 SW_Push, SW18 SW_Push, SW19 SW_Push, SW2 SW_Push, SW20 SW_Push, SW21 SW_Push, SW22 SW_Push, SW23 SW_Push, SW24 SW_Push, SW25 SW_Push, SW26 SW_Push, SW27 SW_Push, SW28 SW_Push, SW29 SW_Push, SW3 SW_Push, SW30 SW_Push, SW31 SW_Push, SW32 SW_Push, SW33 SW_Push, SW34 SW_Push, SW35 SW_Push, SW36 SW_Push, SW37 SW_Push, SW38 SW_Push, SW39 SW_Push, SW4 SW_Push, SW40 RED, SW41 SW_Push, SW42 SW_Push, SW43 SW_Push, SW44 SW_Push, SW45 SW_Push, SW46 SW_Push, SW47 SW_Push, SW48 SW_Push, SW49 SW_Push, SW5 SW_Push, SW50 SW_Push, SW51 SW_Push, SW52 SW_Push, SW53 BLUE, SW54 GREEN, SW55 SW_Push, SW56 SW_Push, SW57 SW_Push, SW58 SW_Push, SW59 SW_Push, SW6 SW_Push, SW60 SW_Push, SW7 SW_Push, SW8 SW_Push, SW9 SW_Push, U1 ATmega32U4-AU

Commit message: Half way through cleaning up keyswitch models and placement
Parts:
- removed U1: ATmega32U4-AU, Package_QFP:TQFP-44_10x10mm_P0.8mm, symbol MCU_Microchip_ATmega:ATmega32U4-AU
- added U1: AT90USB1286-A, Package_QFP:TQFP-64_14x14mm_P0.8mm, symbol MCU_Microchip_AVR:AT90USB1286-A
- D1, D10, D11, D12, D13, D14, D15, D16, D17, D18, D19, D2, D20, D21, D22, D23, D24, D25, D26, D27, D28, D29, D3, D30, D31, D32, D33, D34, D35, D36, D37, D38, D39, D4, D40, D41, D42, D43, D44, D45, D46, D47, D48, D49, D5, D50, D51, D52, D53, D54, D55, D56, D57, D58, D59, D6, D60, D7, D8, D9: footprint Diode_SMD:D_1206_3216Metric_Pad1.42x1.75mm_HandSolder -> Diode_SMD:D_1206_3216Metric
Connections:
- new net: U1.21 (VCC), U1.52 (VCC)
- new net: U1.22 (GND), U1.53 (GND), U1.63 (GND)
Other:
- moved on the sheet: D1, D10, D11, D12, D13, D14, D15, D16, D17, D18, D19, D2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

Commit message: Test commit
Parts:
- removed U1: AT90USB1286-A, Package_QFP:TQFP-64_14x14mm_P0.8mm, symbol MCU_Microchip_AVR:AT90USB1286-A
- added U?: ATmega32U4-A, Package_QFP:TQFP-44_10x10mm_P0.8mm, symbol MCU_Microchip_ATmega:ATmega32U4-A
Connections:
- new net: U?.14 (VCC), U?.34 (VCC)
- new net: U?.24 (AVCC), U?.44 (AVCC)
- new net GND: U?.15 (GND), U?.23 (GND), U?.35 (GND), U?.43 (GND), U?.5 (UGND)
Other:
- moved on the sheet: D1, D10, D11, D12, D13, D14, D15, D16, D17, D18, D19, D2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

Commit message: Cleanup, reference designs and sticking with atmega
Parts:
- added C1, C4, C5, C6, C7: C, Capacitor_SMD:C_0603_1608Metric, symbol Device:C
- added C2, C3: 22p, Capacitor_SMD:C_0603_1608Metric, symbol Device:C
- added J1: USB_C_Receptacle_USB2.0, USB:GCT_USB4055-30-A, symbol Connector:USB_C_Receptacle_USB2.0
- added R1, R2: 10k, Resistor_SMD:R_0603_1608Metric, symbol Device:R
- added R3, R4: 22R, Resistor_SMD:R_0603_1608Metric, symbol Device:R
- added SW61: SW_Push, Button_Switch_SMD:Panasonic_EVQPUJ_EVQPUA, symbol Switch:SW_Push
- added Y1: Crystal_GND24, Crystal:Crystal_SMD_0603-4Pin_6.0x3.5mm, symbol Device:Crystal_GND24
- gave numbers to parts that had none: 1
Connections:
- net ROW6 is gone; now on net ROW5: D20.1 (K), D25.1 (K), D46.1 (K), D5.1 (K), D51.1 (K), D55.1 (K), D59.1 (K), D60.1 (K)
- net COL0: now also U1.37 (PF6)
- net COL1: now also U1.8 (PB0)
- net COL10: now also U1.25 (PD4)
- net COL11: now also U1.22 (PD5)
- net COL2: now also U1.40 (PF1)
- net COL3: now also U1.19 (PD1)
- net COL4: now also U1.32 (PC7)
- net COL5: now also U1.31 (PC6)
- net COL6: now also U1.12 (PB7)
- net COL7: now also U1.30 (PB6)
- net COL8: now also U1.27 (PD7)
- net COL9: now also U1.26 (PD6)
- net GND: now also C1.2, C2.2, C3.2, C4.2, C5.2, C6.2, C7.2, J1.A1 (GND), J1.A12 (GND), J1.B1 (GND), J1.B12 (GND), R2.2, SW61.1, Y1.2, Y1.4
- net ROW0: now also U1.1 (PE6)
- net ROW1: now also U1.29 (PB5)
- net ROW3: now also D14.1 (K), D19.1 (K), D24.1 (K), D29.1 (K), D33.1 (K), D37.1 (K), D4.1 (K), D41.1 (K), D45.1 (K), D50.1 (K), D54.1 (K), D9.1 (K), U1.39 (PF4); no longer D13.1 (K), D18.1 (K), D23.1 (K), D28.1 (K), D3.1 (K), D32.1 (K), D36.1 (K), D40.1 (K), D44.1 (K), D49.1 (K), D53.1 (K), D58.1 (K), D8.1 (K)
- net ROW4: now also D10.1 (K), D15.1 (K), U1.38 (PF5); no longer D14.1 (K), D19.1 (K), D24.1 (K), D29.1 (K), D33.1 (K), D37.1 (K), D4.1 (K), D41.1 (K), D45.1 (K), D50.1 (K), D54.1 (K), D9.1 (K)
- net ROW5: now also U1.28 (PB4); no longer D10.1 (K), D15.1 (K)
- net MOSI: now reaches U1.10 (PB2)
- net MISO: now reaches U1.11 (PB3)
- net Reset: now reaches U1.13 (~{RESET})
- net Reset: now also R1.1, SW61.2
- net +5V: now reaches U1.14 (VCC), U1.34 (VCC)
- net +5V: now also U1.2 (UVCC), U1.24 (AVCC), U1.44 (AVCC), U1.7 (VBUS), C4.1, C5.1, C6.1, C7.1, J1.A4 (VBUS), J1.A9 (VBUS), J1.B4 (VBUS), J1.B9 (VBUS), R1.2
- net XTAL2: now reaches U1.16 (XTAL2)
- net XTAL2: now also C2.1, Y1.3
- net XTAL1: now reaches U1.17 (XTAL1)
- net XTAL1: now also C3.1, Y1.1
- net at U1.3 (D-): now also R4.2
- net at U1.33 (~{HWB}/PE2): now also R2.1
- net ROW2: now reaches U1.36 (PF7)
- net ROW2: now also D13.1 (K), D18.1 (K), D23.1 (K), D28.1 (K), D3.1 (K), D32.1 (K), D36.1 (K), D40.1 (K), D44.1 (K), D49.1 (K), D53.1 (K), D58.1 (K), D8.1 (K)
- net at U1.4 (D+): now also R3.2
- net at U1.6 (UCAP): now also C1.1
- net SCK: now reaches U1.9 (PB1)
- new net D+: J1.A6 (D+), J1.B6 (D+), R3.1
- new net D-: J1.A7 (D-), J1.B7 (D-), R4.1
- no-connect marks 0 -> 3
Other:
- moved on the sheet: U1

Commit message: Rought placement of mounting holes + routing
Connections:
- net COL0: now also U1.30 (PB6); no longer U1.37 (PF6)
- net COL1: now also U1.31 (PC6); no longer U1.8 (PB0)
- net COL10: now also U1.20 (PD2); no longer U1.25 (PD4)
- net COL11: now also U1.21 (PD3); no longer U1.22 (PD5)
- net COL12: now also U1.22 (PD5)
- net COL2: now also U1.32 (PC7); no longer U1.40 (PF1)
- net COL3: now also U1.36 (PF7); no longer U1.19 (PD1)
- net COL4: now also U1.37 (PF6); no longer U1.32 (PC7)
- net COL5: now also U1.8 (PB0); no longer U1.31 (PC6)
- net COL6: now also U1.41 (PF0); no longer U1.12 (PB7)
- net COL7: now also U1.12 (PB7); no longer U1.30 (PB6)
- net COL8: now also U1.18 (PD0); no longer U1.27 (PD7)
- net COL9: now also U1.19 (PD1); no longer U1.26 (PD6)
- net ROW0: now also U1.25 (PD4); no longer U1.1 (PE6)
- net ROW1: now also U1.26 (PD6); no longer U1.29 (PB5)
- net ROW2: now also U1.27 (PD7); no longer U1.36 (PF7)
- net ROW3: now also U1.28 (PB4); no longer U1.39 (PF4)
- net ROW4: now also D20.1 (K), D25.1 (K), D46.1 (K), D5.1 (K), D51.1 (K), D55.1 (K), D59.1 (K), D60.1 (K), U1.29 (PB5); no longer U1.38 (PF5)
- removed net ROW5: D20.1 (K), D25.1 (K), D46.1 (K), D5.1 (K), D51.1 (K), D55.1 (K), D59.1 (K), D60.1 (K), U1.28 (PB4)
- no-connect marks 3 -> 6
Other:
- moved on the sheet: C4, C5
