File: Hardware/PCB/Orthodox.kicad_sch (KiCad schematic)
At the start: 135 parts, among them J1 USB_C_Receptacle_USB2.0, SW1 SW_Push, SW10 SW_Push, SW11 SW_Push, SW12 SW_Push, SW13 SW_Push, SW14 SW_Push, SW15 SW_Push, SW16 SW_Push, SW17 SW_Push, SW18 SW_Push, SW19 SW_Push, SW2 SW_Push, SW20 SW_Push, SW21 SW_Push, SW22 SW_Push, SW23 SW_Push, SW24 SW_Push, SW25 SW_Push, SW26 SW_Push, SW27 SW_Push, SW28 SW_Push, SW29 SW_Push, SW3 SW_Push, SW30 SW_Push, SW31 SW_Push, SW32 SW_Push, SW33 SW_Push, SW34 SW_Push, SW35 SW_Push, SW36 SW_Push, SW37 SW_Push, SW38 SW_Push, SW39 SW_Push, SW4 SW_Push, SW40 RED, SW41 SW_Push, SW42 SW_Push, SW43 SW_Push, SW44 SW_Push, SW45 SW_Push, SW46 SW_Push, SW47 SW_Push, SW48 SW_Push, SW49 SW_Push, SW5 SW_Push, SW50 SW_Push, SW51 SW_Push, SW52 SW_Push, SW53 BLUE, SW54 GREEN, SW55 SW_Push, SW56 SW_Push, SW57 SW_Push, SW58 SW_Push, SW59 SW_Push, SW6 SW_Push, SW60 SW_Push, SW61 SW_Push, SW7 SW_Push, SW8 SW_Push, SW9 SW_Push, U1 ATmega32U4-A, Y1 Crystal_GND24

Commit message: Edited folders to be clearer, added 1st draft of coil to WSAD + ARROW.
Parts:
- added J2: Coil, symbol Connector:Conn_01x02_Female
- SW16, SW27, SW28, SW29, SW50, SW58, SW59, SW60: footprint Switch_Keyboard_Kailh:SW_Kailh_Choc_V1_1.00u -> Switch_Keyboard_Kailh:SW_Kailh_Choc_V1_1.00u_coil
Changed lines of the file:
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@@
     (property "Reference" "SW50" (id 0) (at 250.19 95.631 0))
     (property "Value" "SW_Push" (id 1) (at 250.19 97.9424 0))
-    (property "Footprint" "Switch_Keyboard_Kailh:SW_Kailh_Choc_V1_1.00u" (id 2) (at 250.19 97.79 0)
+    (property "Footprint" "Switch_Keyboard_Kailh:SW_Kailh_Choc_V1_1.00u_coil" (id 2) (at 250.19 97.79 0)
       (effects (font (size 1.27 1.27)) hide)
     )
@@
     (property "Reference" "SW27" (id 0) (at 59.69 75.311 0))
     (property "Value" "SW_Push" (id 1) (at 59.69 77.6224 0))
-    (property "Footprint" "Switch_Keyboard_Kailh:SW_Kailh_Choc_V1_1.00u" (id 2) (at 59.69 77.47 0)
+    (property "Footprint" "Switch_Keyboard_Kailh:SW_Kailh_Choc_V1_1.00u_coil" (id 2) (at 59.69 77.47 0)
       (effects (font (size 1.27 1.27)) hide)
     )
@@
     (property "Reference" "SW16" (id 0) (at 78.74 54.991 0))
     (property "Value" "SW_Push" (id 1) (at 78.74 57.3024 0))
-    (property "Footprint" "Switch_Keyboard_Kailh:SW_Kailh_Choc_V1_1.00u" (id 2) (at 78.74 57.15 0)
+    (property "Footprint" "Switch_Keyboard_Kailh:SW_Kailh_Choc_V1_1.00u_coil" (id 2) (at 78.74 57.15 0)
       (effects (font (size 1.27 1.27)) hide)
     )
@@
     (property "Reference" "SW28" (id 0) (at 78.74 75.311 0))
     (property "Value" "SW_Push" (id 1) (at 78.74 77.6224 0))
-    (property "Footprint" "Switch_Keyboard_Kailh:SW_Kailh_Choc_V1_1.00u" (id 2) (at 78.74 77.47 0)
+    (property "Footprint" "Switch_Keyboard_Kailh:SW_Kailh_Choc_V1_1.00u_coil" (id 2) (at 78.74 77.47 0)
       (effects (font (size 1.27 1.27)) hide)
     )
@@
     (property "Reference" "SW58" (id 0) (at 231.14 131.191 0))
     (property "Value" "SW_Push" (id 1) (at 231.14 133.5024 0))
-    (property "Footprint" "Switch_Keyboard_Kailh:SW_Kailh_Choc_V1_1.00u" (id 2) (at 231.14 133.35 0)
+    (property "Footprint" "Switch_Keyboard_Kailh:SW_Kailh_Choc_V1_1.00u_coil" (id 2) (at 231.14 133.35 0)
       (effects (font (size 1.27 1.27)) hide)
     )
@@
     (property "Reference" "SW29" (id 0) (at 97.79 75.311 0))
     (property "Value" "SW_Push" (id 1) (at 97.79 77.6224 0))
-    (property "Footprint" "Switch_Keyboard_Kailh:SW_Kailh_Choc_V1_1.00u" (id 2) (at 97.79 77.47 0)
+    (property "Footprint" "Switch_Keyboard_Kailh:SW_Kailh_Choc_V1_1.00u_coil" (id 2) (at 97.79 77.47 0)
       (effects (font (size 1.27 1.27)) hide)
     )
@@
     (property "Reference" "SW59" (id 0) (at 250.19 131.191 0))
     (property "Value" "SW_Push" (id 1) (at 250.19 133.5024 0))
-    (property "Footprint" "Switch_Keyboard_Kailh:SW_Kailh_Choc_V1_1.00u" (id 2) (at 250.19 133.35 0)
+    (property "Footprint" "Switch_Keyboard_Kailh:SW_Kailh_Choc_V1_1.00u_coil" (id 2) (at 250.19 133.35 0)
       (effects (font (size 1.27 1.27)) hide)
     )
@@
     (property "Reference" "SW60" (id 0) (at 269.24 131.191 0))
     (property "Value" "SW_Push" (id 1) (at 269.24 133.5024 0))
-    (property "Footprint" "Switch_Keyboard_Kailh:SW_Kailh_Choc_V1_1.00u" (id 2) (at 269.24 133.35 0)
+    (property "Footprint" "Switch_Keyboard_Kailh:SW_Kailh_Choc_V1_1.00u_coil" (id 2) (at 269.24 133.35 0)
       (effects (font (size 1.27 1.27)) hide)
     )
@@
     )
     (property "Datasheet" "~" (id 3) (at 274.32 142.24 0)
+      (effects (font (size 1.27 1.27)) hide)
+    )
+    (pin "1")
+    (pin "2")
+  )
+  (symbol (lib_id "Connector:Conn_01x02_Female") (at 217.17 182.88 270) (unit 1)
+    (in_bom yes) (on_board yes) (fields_autoplaced)
+    (property "Reference" "J2" (id 0) (at 218.44 180.9749 90)
+      (effects (font (size 1.27 1.27)) (justify left))
+    )
+    (property "Value" "Coil" (id 1) (at 218.44 183.5149 90)
+      (effects (font (size 1.27 1.27)) (justify left))
+    )
+    (property "Footprint" "" (id 2) (at 217.17 182.88 0)
+      (effects (font (size 1.27 1.27)) hide)
+    )
+    (property "Datasheet" "~" (id 3) (at 217.17 182.88 0)
       (effects (font (size 1.27 1.27)) hide)
     )
@@
       (reference "J1") (unit 1) (value "USB_C_Receptacle_USB2.0") (footprint "USB:GCT_USB4055-30-A")
     )
+    (path "/02520595-683f-405b-b632-abaecde555b7"
+      (reference "J2") (unit 1) (value "Coil") (footprint "")
+    )
     (path "/13513b6d-df2b-4cc8-aa13-36ec19259a60"
       (reference "R1") (unit 1) (value "10k") (footprint "Resistor_SMD:R_0603_1608Metric")
@@
     )
     (path "/00000000-0000-0000-0000-00006179071e"
-      (reference "SW16") (unit 1) (value "SW_Push") (footprint "Switch_Keyboard_Kailh:SW_Kailh_Choc_V1_1.00u")
+      (reference "SW16") (unit 1) (value "SW_Push") (footprint "Switch_Keyboard_Kailh:SW_Kailh_Choc_V1_1.00u_coil")
     )
     (path "/00000000-0000-0000-0000-000061793b1a"
@@
     )
     (path "/00000000-0000-0000-0000-00006178dd92"
-      (reference "SW27") (unit 1) (value "SW_Push") (footprint "Switch_Keyboard_Kailh:SW_Kailh_Choc_V1_1.00u")
+      (reference "SW27") (unit 1) (value "SW_Push") (footprint "Switch_Keyboard_Kailh:SW_Kailh_Choc_V1_1.00u_coil")
     )
     (path "/00000000-0000-0000-0000-00006179072a"
-      (reference "SW28") (unit 1) (value "SW_Push") (footprint "Switch_Keyboard_Kailh:SW_Kailh_Choc_V1_1.00u")
+      (reference "SW28") (unit 1) (value "SW_Push") (footprint "Switch_Keyboard_Kailh:SW_Kailh_Choc_V1_1.00u_coil")
     )
     (path "/00000000-0000-0000-0000-000061793b26"
-      (reference "SW29") (unit 1) (value "SW_Push") (footprint "Switch_Keyboard_Kailh:SW_Kailh_Choc_V1_1.00u")
+      (reference "SW29") (unit 1) (value "SW_Push") (footprint "Switch_Keyboard_Kailh:SW_Kailh_Choc_V1_1.00u_coil")
     )
     (path "/00000000-0000-0000-0000-00006179c887"
@@
     )
     (path "/00000000-0000-0000-0000-00006178c30e"
-      (reference "SW50") (unit 1) (value "SW_Push") (footprint "Switch_Keyboard_Kailh:SW_Kailh_Choc_V1_1.00u")
+      (reference "SW50") (unit 1) (value "SW_Push") (footprint "Switch_Keyboard_Kailh:SW_Kailh_Choc_V1_1.00u_coil")
     )
     (path "/00000000-0000-0000-0000-00006178ddaa"
@@
     )
     (path "/00000000-0000-0000-0000-000061790748"
-      (reference "SW58") (unit 1) (value "SW_Push") (footprint "Switch_Keyboard_Kailh:SW_Kailh_Choc_V1_1.00u")
+      (reference "SW58") (unit 1) (value "SW_Push") (footprint "Switch_Keyboard_Kailh:SW_Kailh_Choc_V1_1.00u_coil")
     )
     (path "/00000000-0000-0000-0000-000061793b44"
-      (reference "SW59") (unit 1) (value "SW_Push") (footprint "Switch_Keyboard_Kailh:SW_Kailh_Choc_V1_1.00u")
+      (reference "SW59") (unit 1) (value "SW_Push") (footprint "Switch_Keyboard_Kailh:SW_Kailh_Choc_V1_1.00u_coil")
     )
     (path "/00000000-0000-0000-0000-00006179c8a5"
-      (reference "SW60") (unit 1) (value "SW_Push") (footprint "Switch_Keyboard_Kailh:SW_Kailh_Choc_V1_1.00u")
+      (reference "SW60") (unit 1) (value "SW_Push") (footprint "Switch_Keyboard_Kailh:SW_Kailh_Choc_V1_1.00u_coil")
     )
     (path "/3b0bf36b-f5e1-40fa-931a-45165d475f4e"
